File: ATtiny prog board/ATtiny prog board.brd (EAGLE design)
At the start: 17.8 x 21.6 mm, 10 parts

Commit message: added some info to silk screen
Other:
- board text added: "+"
Changed lines of the file:
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@@
 <wire x1="15.987359375" y1="21.58" x2="1.78899375" y2="21.58" width="0" layer="20"/>
 <wire x1="1.78899375" y1="21.58" x2="0" y2="19.79100625" width="0" layer="20" curve="90"/>
+<text x="15.875" y="12.065" size="1.778" layer="25">+</text>
 </plain>
 <attributes>
@@
 <attribute name="PROD_ID" value="IC-09445" x="6.35" y="7.62" size="1.778" layer="27" display="off"/>
 <attribute name="VALUE" x="3.175" y="6.985" size="1.27" layer="27" ratio="10"/>
-<attribute name="NAME" x="1.5875" y="7.62" size="0.8128" layer="25" ratio="10" rot="R90"/>
-</element>
-<element name="ISP" library="SparkFun-Connectors" package="2X3" value="" x="16.51" y="19.05" rot="R180"/>
+<attribute name="NAME" x="5.3975" y="6.6675" size="0.8128" layer="25" ratio="10" rot="R90"/>
+</element>
+<element name="ISP" library="SparkFun-Connectors" package="2X3" value="" x="16.51" y="19.05" smashed="yes" rot="R180">
+<attribute name="NAME" x="17.4625" y="14.9225" size="1.27" layer="25" ratio="10" rot="R180"/>
+<attribute name="VALUE" x="17.78" y="22.225" size="1.27" layer="27" rot="R180"/>
+</element>
 <element name="JP1" library="SparkFun-Connectors" package="1X06" value="" x="15.24" y="1.27" rot="R180">
 <attribute name="PROD_ID" value="CONN-08437" x="15.24" y="1.27" size="1.778" layer="27" rot="R180" display="off"/>
@@
 </polygon>
 <via x="13.0175" y="13.97" extent="1-16" drill="0.6"/>
+<via x="2.2225" y="13.335" extent="1-16" drill="0.6"/>
+<via x="0.9525" y="2.54" extent="1-16" drill="0.6"/>
+<via x="11.43" y="2.54" extent="1-16" drill="0.6"/>
+<via x="3.81" y="2.54" extent="1-16" drill="0.6"/>
 </signal>
 <signal name="PB0/MOSI">
