File: voltage inverter/EAGLE (remake)/ICL7660.brd (EAGLE design)
At the start: 15.2 x 11.4 mm, 5 parts, among them IC1 ICL7660

Commit message: updated brd & images
Routing:
- net GND: vias 0 -> 4
Changed lines of the file:
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@@
 <wire x1="12.065" y1="6.985" x2="13.0175" y2="7.9375" width="0.4064" layer="1"/>
 <wire x1="13.0175" y1="7.9375" x2="13.0175" y2="8.407" width="0.4064" layer="1"/>
+<via x="7.62" y="8.5725" extent="1-16" drill="0.6"/>
+<via x="12.065" y="10.16" extent="1-16" drill="0.6"/>
+<via x="14.2875" y="2.8575" extent="1-16" drill="0.6"/>
+<via x="10.795" y="2.54" extent="1-16" drill="0.6"/>
 </signal>
 <signal name="N$1">
