File: DBx breakout/DA-15_DB-9_DE-15.sch (EAGLE design)
At the start: 3 parts

Commit message: updated board
Parts:
- added RAIL1, RAIL2: M02PTH, SparkFun-Connectors:M02PTH
- DE-15: device adafruit:F15HDV -> con-subd:HF15H
Connections:
- new net SHIELD: RAIL1.1, RAIL1.2, RAIL2.1, RAIL2.2
Other:
- moved on the sheet: HEADER
